Commit message: added new urdf model

File: youbot_description/robots/youbot.urdf.xacro (robot description, xacro)
@@ -12,6 +12,6 @@
   <!-- youbot plate -->
   <!--xacro:include filename="$(find youbot_description)/urdf/youbot_plate/plate.urdf.xacro" /-->
-  <!-- youbot plate V2 -->
-  <xacro:include filename="$(find youbot_description)/urdf/youbot_plateV2/plateV2.urdf.xacro" />
+  <!-- youbot assembly -->
+  <xacro:include filename="$(find youbot_description)/urdf/YouBot_Assembly/YouBot_Assembly.urdf.xacro" />
   <!-- youbot arm -->
   <xacro:include filename="$(find youbot_description)/urdf/youbot_arm/arm.urdf.xacro"/>
@@ -34,9 +34,9 @@
   <!-- foot for arm-->
   <xacro:youbot_base name="base"/>
-  <xacro:youbot_plateV2 name="youbot_plateV2" parent="base_link">
-    <origin xyz="0 0 0.06" rpy="1.5707963267949 0 0" />
-  </xacro:youbot_plateV2>
+  <xacro:YouBot_Assembly name="YouBot_Assembly" parent="base_link">
+    <origin xyz="0 0 -0.093" rpy="0 0 0" />
+  </xacro:YouBot_Assembly>
   <xacro:youbot_arm name="arm" parent="base_link">
-    <origin xyz="0.2 0.08 0.1" rpy="0 0 1.5707963267949" />
+    <origin xyz="0.2 0.09 0.093" rpy="0 0 1.5707963267949" />
   </xacro:youbot_arm>
   <xacro:youbot_gripper name="gripper" parent="arm_link_5">
@@ -44,6 +44,10 @@
   </xacro:youbot_gripper>
   <!-- base laser front -->
-  <xacro:hokuyo_urg04_laser name="base_laser_front" parent="base" ros_topic="scan_front" update_rate="10" min_angle="-1.57" max_angle="1.57">
-    <origin xyz="0.3 0 -0.03" rpy="0 0 0"/>
+  <xacro:hokuyo_urg04_laser name="base_laser_front" parent="base" ros_topic="scan_front" update_rate="10" min_angle="-2.35" max_angle="2.35">
+    <origin xyz="0.25 -0.15 0.06" rpy="3.14 0 0.785398163397448"/>
+  </xacro:hokuyo_urg04_laser>
+ <!-- base laser back -->
+  <xacro:hokuyo_urg04_laser name="base_laser_back" parent="base" ros_topic="scan_front" update_rate="10" min_angle="-2.35" max_angle="2.35">
+    <origin xyz="-0.25 0.15 0.06" rpy="3.14 0 -0.785398163397448"/>
   </xacro:hokuyo_urg04_laser>
 </robot>

File: youbot_description/urdf/YouBot_Assembly/YouBot_Assembly.urdf.xacro (robot description, xacro)
@@ -4,5 +4,5 @@
        xmlns:interface="http://playerstage.sourceforge.net/gazebo/xmlschema/#interface"
        xmlns:xacro="http://ros.org/wiki/xacro">
-	<xacro:macro name="YouBot_Assembly_URDF" params="parent name *origin">
+	<xacro:macro name="YouBot_Assembly" params="parent name *origin">
 		<joint name="${name}_joint" type="fixed" >
 			<insert_block name="origin" />
@@ -23,5 +23,5 @@
 			</inertial>
 			<visual>
-				<origin xyz="1.5707963267949 0 0" rpy="0 0 0" />
+				<origin xyz="0 0 0" rpy="1.5707963267949 0 3.14" />
 				<geometry>
 					<mesh filename="package://youbot_description/meshes/YouBot_Assembly/YouBot_Assembly.STL" />
@@ -30,5 +30,5 @@
 			</visual>
 			<collision>
-				<origin xyz="0 0 0" rpy="1.5707963267949 0 0" />
+				<origin xyz="0 0 0" rpy="1.5707963267949 0 3.14" />
 				<geometry>
 					<mesh filename="package://youbot_description/meshes/YouBot_Assembly/YouBot_Assembly.STL" />
